File: Servo Tester.kicad_sch (KiCad schematic)
At the start: 0 parts

Commit message: Added Components to Schematic
Parts:
- added C1: C, symbol Device:C
- added D1: 1N4148, Diode_THT:D_DO-35_SOD27_P7.62mm_Horizontal, symbol Diode:1N4148
- added D2: LED, symbol Device:LED
- added J1: Conn_01x02_Pin, symbol Connector:Conn_01x02_Pin
- added J2: Conn_01x03_Pin, symbol Connector:Conn_01x03_Pin
- added R1, R2, R3: R, symbol Device:R
- added RV1: R_Potentiometer, symbol Device:R_Potentiometer
- added U1: NE555P, Package_DIP:DIP-8_W7.62mm, symbol Timer:NE555P
